File: schems/electrical/pHmeter.kicad_sch (KiCad schematic)
At the start: 23 parts, among them J1 Screw_Terminal_01x02, J2 Conn_01x04, J3 Conn_01x02, J4 Screw_Terminal_01x02, J5 SD_Card, J6 Conn_01x03_Pin, J7 Conn_01x03_Pin, K1 FINDER-36.11, K2 FINDER-36.11, Q1 2N7000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

Commit message: update schem
Parts:
- added J8, J9: Screw_Terminal_01x03, symbol Connector:Screw_Terminal_01x03
- added Q4: BC547, Package_TO_SOT_THT:TO-92_Inline, symbol Transistor_BJT:BC547
- added R5: 4,7K, Resistor_THT:R_Axial_DIN0207_L6.3mm_D2.5mm_P10.16mm_Horizontal, symbol Device:R
- added SW4, SW5, SW6: SW_Push, Button_Switch_THT:SW_PUSH_6mm_H8mm, symbol Switch:SW_Push
Connections:
- net +9V is gone; now on net +12V: A1.30 (VIN), SW3.1 (A)
- net +BATT: no longer SW3.2 (B)
- net Data: now also A1.10 (D7); no longer A1.7 (D4)
- net EC_vcc: now also A1.12 (D9), R4.1; no longer A1.9 (D6)
- net GND: now also Q3.3 (E), Q4.3 (E), SW4.1, SW5.1, SW6.1
- net Ph_vcc: now also A1.11 (D8), R5.1; no longer A1.8 (D5)
- net SD_CS: now also A1.13 (D10)
- net at Q3.1 (C): now also D2.2 (A), K2.A2
- net at Q3.2 (B): now also R4.2
- net +12V: now reaches D2.1 (K)
- net +12V: now also D1.1 (K), K1.A1, K2.A1
- net at K2.11: now also J8.2 (Pin_2)
- net at K2.12: now also J8.3 (Pin_3)
- net at K2.14: now also J8.1 (Pin_1)
- net at D1.2 (A): now also K1.A2, Q4.1 (C)
- net at K1.11: now also J9.2 (Pin_2)
- net at K1.12: now also J9.3 (Pin_3)
- net at K1.14: now also J9.1 (Pin_1)
- new net: A1.7 (D4), SW4.2
- new net: A1.8 (D5), SW5.2
- new net: A1.9 (D6), SW6.2
- new net: Q4.2 (B), R5.2
- new net VDC: SW3.2 (B)
Other:
- moved on the sheet: D1, D2, J5, K1, K2, Q3, R4, SW1, SW2
